File: PCB/PCB.kicad_sch (KiCad schematic)
At the start: 34 parts, among them J1 RJ45, J2 RJ45, U1 Pico, U2 LM358, U3 LM358

Commit message: Schematic and readme cleanup
Other:
- note added: "1uF & 32k is 32 ms Time Constant"
- note added: "CT Burden"
- note added: "Cap Touch"
- note added: "LED"
- note removed: "1uF & 32k is 32ms TC"
- note removed: "Burden"
Changed lines of the file:
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@@
     (stroke (width 0) (type default))
   )
-  (text "Unused\n" (at 144.78 22.86 0)
-    (effects (font (size 1.27 1.27)) (justify left bottom))
+  (text "Unused\n" (at 166.37 25.4 0)
+    (effects (font (size 3 3)) (justify left bottom))
   )
-  (text "1uF & 32k is 32ms TC\n\n" (at 173.99 77.47 0)
-    (effects (font (size 1.27 1.27)) (justify left bottom))
+  (text "1uF & 32k is 32 ms\nTime Constant\n\n" (at 172.72 82.55 0)
+    (effects (font (size 2 2)) (justify left bottom))
   )
-  (text "Ideal Diode Peak Dector with Gain = 3.2" (at 179.07 48.26 0)
-    (effects (font (size 1.27 1.27)) (justify left bottom))
+  (text "Ideal Diode Peak Dector with Gain = 3.2" (at 167.64 41.91 0)
+    (effects (font (size 3 3)) (justify left bottom))
   )
-  (text "Burden" (at 153.67 62.23 0)
-    (effects (font (size 1.27 1.27)) (justify left bottom))
+  (text "LED\n\n" (at 83.82 129.54 0)
+    (effects (font (size 4 4)) (justify left bottom))
   )
-  (text "50A / 1600 * 30 Ohms = 0.94 V\n" (at 168.91 96.52 0)
-    (effects (font (size 1.27 1.27)) (justify left bottom))
+  (text "CT\nBurden" (at 142.24 72.39 0)
+    (effects (font (size 2 2)) (justify left bottom))
+  )
+  (text "50A / 1600 * 30 Ohms = 0.94 V\n" (at 168.91 99.06 0)
+    (effects (font (size 3 3)) (justify left bottom))
+  )
+  (text "Cap Touch\n" (at 64.77 88.9 0)
+    (effects (font (size 4 4)) (justify left bottom))
   )
   (text "0.94 V * 3.2 = 3V @ 50A\n\n" (at 198.12 57.15 0)
@@
   )
   (text "Pins 1&2: 1:1600 Current Transformer" (at 168.91 92.71 0)
-    (effects (font (size 1.27 1.27)) (justify left bottom))
+    (effects (font (size 3 3)) (justify left bottom))
   )
   (label "CT1" (at 142.24 93.98 0) (fields_autoplaced)
