File: PCB/PCB.kicad_sch (KiCad schematic)
At the start: 17 parts, among them J1 RJ25, J2 RJ45, U1 Pico, U2 LM358

Commit message: gpio on PCB
Parts:
- added J3: Conn_2Rows-07Pins, Connector_PinHeader_2.54mm:PinHeader_2x07_P2.54mm_Vertical, symbol Connector_Generic:Conn_02x07_Odd_Even
Connections:
- net +5V: now also J3.1 (Pin_1)
- net GND: now also J3.13 (Pin_13), J3.14 (Pin_14)
- net at U1.1 (GPIO0): now also J3.3 (Pin_3)
- net at U1.10 (GPIO7): now also J3.12 (Pin_12)
- net at U1.11 (GPIO8): now also J3.9 (Pin_9)
- net at U1.32 (GPIO27_ADC1): now also J3.11 (Pin_11)
- net at U1.34 (GPIO28_ADC2): now also J3.10 (Pin_10)
- net at U1.36 (3V3): now also J3.2 (Pin_2)
- net at U1.4 (GPIO2): now also J3.4 (Pin_4)
- net at U1.5 (GPIO3): now also J3.5 (Pin_5)
- net at U1.6 (GPIO4): now also J3.6 (Pin_6)
- net at U1.7 (GPIO5): now also J3.7 (Pin_7)
- net at U1.9 (GPIO6): now also J3.8 (Pin_8)
Other:
- note added: "Future"
