File: PCB/PCB.kicad_pcb (KiCad board)
At the start: 4 copper layers, 44.3 x 53.5 mm, 17 parts, among them J1 RJ25, J2 RJ45, U1 Pico, U2 LM358

Commit message: gpio on PCB
Parts:
- added J3: Conn_2Rows-07Pins, Connector_PinHeader_2.54mm:PinHeader_2x07_P2.54mm_Vertical, F.Cu at (112.8, 76.8)
Connections:
- U1 pad 1: unconnected-(U1-GPIO0-Pad1) -> Net-(J3-Pin_3)
- U1 pad 10: unconnected-(U1-GPIO7-Pad10) -> Net-(J3-Pin_12)
- U1 pad 11: unconnected-(U1-GPIO8-Pad11) -> Net-(J3-Pin_9)
- U1 pad 32: unconnected-(U1-GPIO27_ADC1-Pad32) -> Net-(J3-Pin_11)
- U1 pad 34: unconnected-(U1-GPIO28_ADC2-Pad34) -> Net-(J3-Pin_10)
- U1 pad 36: unconnected-(U1-3V3-Pad36) -> Net-(J3-Pin_2)
- U1 pad 4: unconnected-(U1-GPIO2-Pad4) -> Net-(J3-Pin_4)
- U1 pad 5: unconnected-(U1-GPIO3-Pad5) -> Net-(J3-Pin_5)
- U1 pad 6: unconnected-(U1-GPIO4-Pad6) -> Net-(J3-Pin_6)
- U1 pad 7: unconnected-(U1-GPIO5-Pad7) -> Net-(J3-Pin_7)
- U1 pad 9: unconnected-(U1-GPIO6-Pad9) -> Net-(J3-Pin_8)
Routing:
- net Net-(J3-Pin_11): track 0.00 -> 33.8 mm, vias 0 -> 1
- net Net-(J3-Pin_10): track 0.00 -> 29.3 mm, vias 0 -> 1
- net +5V: track 53.1 -> 79.8 mm, vias 1 -> 2
- net Net-(J3-Pin_2): track 0.00 -> 25.6 mm, vias 0 -> 1
- net Net-(J3-Pin_3): track 0.00 -> 18.8 mm
- net Net-(J3-Pin_9): track 0.00 -> 13.5 mm
- net GND: track 75.7 -> 65.3 mm
- net Net-(J3-Pin_5): track 0.00 -> 9.61 mm
- net Net-(J3-Pin_8): track 0.00 -> 9.47 mm
- net Net-(J3-Pin_7): track 0.00 -> 9.25 mm
- net Net-(J3-Pin_4): track 0.00 -> 7.07 mm
- net Net-(J3-Pin_12): track 0.00 -> 6.71 mm
- net Net-(J3-Pin_6): track 0.00 -> 6.02 mm
